File: KiCAD/Micro LED Array/Micro LED Array.kicad_sch (KiCad schematic)
At the start: 113 parts

Commit message: Driver board connected, add interboard fiducials
Connections:
- net Col1: now also D14.2 (A), D21.2 (A), D28.2 (A), D35.2 (A), D42.2 (A), D49.2 (A), D7.2 (A), H27.1, H28.1; no longer D1.2 (A), D15.2 (A), D22.2 (A), D29.2 (A), D36.2 (A), D43.2 (A), D8.2 (A), H15.1, H16.1
- net Col2: now also D13.2 (A), D20.2 (A), D27.2 (A), D34.2 (A), D41.2 (A), D48.2 (A), D6.2 (A), H25.1, H26.1; no longer D16.2 (A), D2.2 (A), D23.2 (A), D30.2 (A), D37.2 (A), D44.2 (A), D9.2 (A), H17.1, H18.1
- net Col3: now also D12.2 (A), D19.2 (A), D26.2 (A), D33.2 (A), D40.2 (A), D47.2 (A), D5.2 (A), H23.1, H24.1; no longer D10.2 (A), D17.2 (A), D24.2 (A), D3.2 (A), D31.2 (A), D38.2 (A), D45.2 (A), H19.1, H20.1
- net Col5: now also D10.2 (A), D17.2 (A), D24.2 (A), D3.2 (A), D31.2 (A), D38.2 (A), D45.2 (A), H19.1, H20.1; no longer D12.2 (A), D19.2 (A), D26.2 (A), D33.2 (A), D40.2 (A), D47.2 (A), D5.2 (A), H23.1, H24.1
- net Col6: now also D16.2 (A), D2.2 (A), D23.2 (A), D30.2 (A), D37.2 (A), D44.2 (A), D9.2 (A), H17.1, H18.1; no longer D13.2 (A), D20.2 (A), D27.2 (A), D34.2 (A), D41.2 (A), D48.2 (A), D6.2 (A), H25.1, H26.1
- net Col7: now also D1.2 (A), D15.2 (A), D22.2 (A), D29.2 (A), D36.2 (A), D43.2 (A), D8.2 (A), H15.1, H16.1; no longer D14.2 (A), D21.2 (A), D28.2 (A), D35.2 (A), D42.2 (A), D49.2 (A), D7.2 (A), H27.1, H28.1
