File: KiCAD/LED Driver/LED Driver - 400µm spacing/_autosave-LED Driver - 400µm spacing.kicad_sch (KiCad schematic)
At the start: 9 parts, among them U1 LP5868TRKPR, U2 ATtiny3226

Commit message: Add microcontroller
Connections:
- net GND: now also U2.11 (6/PB3)
- no-connect marks 22 -> 21
Changed lines of the file:
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@@
-	)
-	(no_connect
-		(at 228.6 74.93)
 	)
 	(no_connect
@@
 					(unit 1)
 				)
+			)
+		)
+	)
+	(symbol
+		(lib_id "power:GND")
+		(at 228.6 74.93 90)
+		(unit 1)
+		(exclude_from_sim no)
+		(in_bom yes)
+		(on_board yes)
+		(dnp no)
+		(fields_autoplaced yes)
+		(property "Reference" "#PWR010"
+			(at 234.95 74.93 0)
+			(effects
+				(font
+					(size 1.27 1.27)
+				)
+				(hide yes)
+			)
+		)
+		(property "Value" "GND"
+			(at 231.775 74.93 90)
+			(effects
+				(font
+					(size 1.27 1.27)
+				)
+				(justify right)
+			)
+		)
+		(property "Footprint" ""
+			(at 228.6 74.93 0)
+			(effects
+				(font
+					(size 1.27 1.27)
+				)
+				(hide yes)
+			)
+		)
+		(property "Datasheet" ""
+			(at 228.6 74.93 0)
+			(effects
+				(font
+					(size 1.27 1.27)
+				)
+				(hide yes)
+			)
+		)
+		(property "Description" ""
+			(at 228.6 74.93 0)
+			(effects
+				(font
+					(size 1.27 1.27)
+				)
+				(hide yes)
+			)
+		)
+		(pin "1"
+		)
+		(instances
+			(project "LED Driver - 400µm spacing"
+				(path "/333dbdf9-e35a-4a4e-87df-f2105d57feb4"
+					(reference "#PWR010")
+					(unit 1)
+				)
