File: KiCAD/LED Controller/LED Controller.kicad_sch (KiCad schematic)
At the start: 7 parts, among them J1 0525590870, J2 Conn_01x02_Socket, J3 Conn_01x02_Pin, J4 Conn_01x02_Socket, U1 Itsy_Bitsy_32u4

Commit message: minor edits
Parts:
- JP1: now in the parts list
Changed lines of the file:
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@@
 		(unit 1)
 		(exclude_from_sim yes)
-		(in_bom no)
+		(in_bom yes)
 		(on_board yes)
 		(dnp no)
