File: KiCAD/Micro LED Array/Micro LED Array - 400µm spacing.pro/Micro LED Array - 400µm spacing.pro.kicad_sch (KiCad schematic)
At the start: 64 parts

Commit message: minor edits
Parts:
- D1, D10, D11, D12, D13, D14, D15, D16, D17, D18, D19, D2, D20, D21, D22, D23, D24, D25, D26, D27, D28, D29, D3, D30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: Manufacturer Kingbright -> LITEON; Part APG0603SEC-E-TT -> LTST-FC03AD-5A
